Commit message: added gps to sam bot

File: sam_bot_description/src/description/sam_bot_description.urdf (robot description, URDF)
Before this commit: robot sam_bot, 7 links, 6 joints
Links:
- added link gps_link, mass 0.125; collision cylinder length=0.055 radius=0.0508; visual cylinder length=0.055 radius=0.0508
Joints:
- added joint gps_joint: type fixed, parent base_link, child gps_link, origin xyz=-0.0 0 0.18 rpy=0 0 0
